Commit message: change configuration of robot4 xacro file

File: robot_urdf/urdf/robot4.xacro (robot description, xacro)
@@ -115,15 +115,37 @@
     <joint_properties damping="1.0" friction="1.0"/>
   </joint>
-  <link name="camera_link">
+   <link name="camera_link_connection">
 	    <collision>
-	      <origin xyz="0 0 0.025" rpy="0 0 0"/>
+	      <origin xyz="0 0 0.1" rpy="0 0 0"/>
 	      <geometry>
-		<box size="0.05 0.05 0.05"/>
+		<box size="0.1 0.1 0.25"/>
 	      </geometry>
 	    </collision>
 	    <visual>
-	      <origin xyz="0 0 0.025" rpy="0 0 0"/>
+	      <origin xyz="0 0 0.1" rpy="0 0 0"/>
 	      <geometry>
-		<box size="0.05 0.05 0.05"/>
+		<box size="0.05 0.05 0.25"/>
+	      </geometry>
+	      <material name="red">
+		<color rgba="1 0 0 1"/>
+	      </material>
+	    </visual>
+	    <inertial>
+	      <mass value="1e-5" />
+	      <origin xyz="0 0 0" rpy="0 0 0"/>
+	      <inertia ixx="1e-6" ixy="0" ixz="0" iyy="1e-6" iyz="0" izz="1e-6" />
+	    </inertial>
+  </link>
+  <link name="camera_link">
+	    <collision>
+	      <origin xyz="0 0 0" rpy="0 0 0"/>
+	      <geometry>
+		<box size="0.07 0.07 0.07"/>
+	      </geometry>
+	    </collision>
+	    <visual>
+	      <origin xyz="0 0 0" rpy="0 0 0"/>
+	      <geometry>
+		<box size="0.07 0.07 0.07"/>
 	      </geometry>
 	      <material name="red">
@@ -139,7 +161,13 @@
   <joint name="camera_joint" type="fixed">
 	    <axis xyz="0 0 1" />
-	    <origin xyz="0.23 0 0" rpy="0 0 0"/>
-	    <parent link="link_chassis"/>
+	    <origin xyz="0 0 0.27" rpy="0 0 0"/>
+	    <parent link="camera_link_connection"/>
 	    <child link="camera_link"/>
 	 </joint>
+     <joint name="camera_link_joint" type="fixed">
+	    <axis xyz="0 0 1" />
+	    <origin xyz="0.2 0 0.05" rpy="0 0 0"/>
+	    <parent link="link_chassis"/>
+	    <child link="camera_link_connection"/>
+	 </joint>
 </robot>

Commit message: make running the code

File: robot_urdf/urdf/robot4.xacro (robot description, xacro)
@@ -171,3 +171,13 @@
 	    <child link="camera_link_connection"/>
 	 </joint>
+    <transmission name="cam_trans">
+      <type>transmission_interface/SimpleTransmission</type>
+      <joint name="camera_joint">
+      <hardwareInterface>hardwareInterface/EffortJointInterface</hardwareInterface>
+      </joint>
+      <actuator name="motor_cam">
+        <hardwareInterface>hardwareInterface/EffortJointInterface</hardwareInterface>
+        <mechanicalReduction>1</mechanicalReduction>
+      </actuator>
+   </transmission>
 </robot>

Commit message: make camera joint better

File: robot_urdf/urdf/robot4.xacro (robot description, xacro)
@@ -117,13 +117,13 @@
    <link name="camera_link_connection">
 	    <collision>
-	      <origin xyz="0 0 0.1" rpy="0 0 0"/>
+	      <origin xyz="0 0 0.05" rpy="0 0 0"/>
 	      <geometry>
-		<box size="0.1 0.1 0.25"/>
+		<box size="0.05 0.05 0.15"/>
 	      </geometry>
 	    </collision>
 	    <visual>
-	      <origin xyz="0 0 0.1" rpy="0 0 0"/>
+	      <origin xyz="0 0 0.05" rpy="0 0 0"/>
 	      <geometry>
-		<box size="0.05 0.05 0.25"/>
+		<box size="0.05 0.05 0.15"/>
 	      </geometry>
 	      <material name="red">
@@ -161,5 +161,5 @@
   <joint name="camera_joint" type="continuous">
 	    <axis xyz="0 0 1" />
-	    <origin xyz="0 0 0.27" rpy="0 0 0"/>
+	    <origin xyz="0 0 0.15" rpy="0 0 0"/>
 	    <parent link="camera_link_connection"/>
 	    <child link="camera_link"/>

Commit message: edit xacro file

File: robot_urdf/urdf/robot4.xacro (robot description, xacro)
@@ -2,4 +2,5 @@
 <robot xmlns:xacro="http://www.ros.org/wiki/xacro" name="robot4_xacro">
 <xacro:include filename="$(find robot_urdf)/urdf/robot4.gazebo"/>
+<xacro:include filename="$(find robot_urdf)/urdf/materials.xacro"/>
 	<xacro:property name="length_wheel" value="0.04" />
 	<xacro:property name="radius_wheel" value="0.1" />
@@ -16,29 +17,5 @@
      	</geometry>
 	</xacro:macro>
-  <material name="black">
-    <color rgba="0.0 0.0 0.0 1.0"/>
-  </material>
-  <material name="blue">
-    <color rgba="0.203125 0.23828125 0.28515625 1.0"/>
-  </material>
-  <material name="green">
-    <color rgba="0.0 0.8 0.0 1.0"/>
-  </material>
-  <material name="grey">
-    <color rgba="0.2 0.2 0.2 1.0"/>
-  </material>
-  <material name="orange">
-    <color rgba="1.0 0.423529411765 0.0392156862745 1.0"/>
-  </material>
-  <material name="brown">
-    <color rgba="0.870588235294 0.811764705882 0.764705882353 1.0"/>
-  </material>
-  <material name="red">
-    <color rgba="0.80078125 0.12890625 0.1328125 1.0"/>
-  </material>
-  <material name="white">
-    <color rgba="1.0 1.0 1.0 1.0"/>
-  </material>
-	  <link name="link_chassis">
+	<link name="link_chassis">
     <!-- pose and inertial -->
     <pose>0 0 0.1 0 0 0</pose>
