Commit message: add wheels in urdf

File: urdf/robot2.urdf (robot description, URDF)
Before this commit: robot diff_robot, 8 links, 7 joints
Links:
- removed link caster_wheel
- removed link left_wheel
- removed link right_wheel
- added link front_left_wheel, mass 0.5; collision cylinder length=0.036 radius=0.04; visual mesh filename=package://rosbot_description/meshes/wheel.stl scale=0.001 0.001 0.001
- added link front_right_wheel, mass 0.5; collision cylinder length=0.036 radius=0.04; visual mesh filename=package://rosbot_description/meshes/wheel.stl scale=0.001 0.001 0.001
- added link rear_left_wheel, mass 0.5; collision cylinder length=0.036 radius=0.04; visual mesh filename=package://rosbot_description/meshes/wheel.stl scale=0.001 0.001 0.001
- added link rear_right_wheel, mass 0.5; collision cylinder length=0.036 radius=0.04; visual mesh filename=package://rosbot_description/meshes/wheel.stl scale=0.001 0.001 0.001
Joints:
- removed joint caster_wheel_joint
- removed joint left_wheel_joint
- removed joint right_wheel_joint
- added joint front_left_wheel_hinge: type continuous, parent body_link, child front_left_wheel, origin xyz=0.05 0.11 0 rpy=0 0 0, axis 0 1 0, limit effort=1 velocity=10
- added joint front_right_wheel_hinge: type continuous, parent body_link, child front_right_wheel, origin xyz=0.05 -0.11 0 rpy=0 0 0, axis 0 1 0, limit effort=1 velocity=10
- added joint rear_left_wheel_hinge: type continuous, parent body_link, child rear_left_wheel, origin xyz=-0.055 0.11 0 rpy=0 0 0, axis 0 1 0, limit effort=1 velocity=10
- added joint rear_right_wheel_hinge: type continuous, parent body_link, child rear_right_wheel, origin xyz=-0.055 -0.11 0 rpy=0 0 0, axis 0 1 0, limit effort=1 velocity=10

Commit message: update urdf

File: urdf/robot2.urdf (robot description, URDF)
Before this commit: robot diff_robot, 9 links, 8 joints
Joints:
- joint front_left_wheel_hinge: parent body_link -> base_link
- joint front_right_wheel_hinge: parent body_link -> base_link
- joint rear_left_wheel_hinge: parent body_link -> base_link
- joint rear_right_wheel_hinge: parent body_link -> base_link
